Commit message: Add namespace to wheels and sensors link

File: urdf/doogie_sensors.xacro (robot description, xacro)
@@ -3,6 +3,7 @@
     <!-- Includes -->
     <xacro:include filename="$(find doogie_description)/urdf/acessories/ir_sensor.xacro"/>
+    <!-- ir_sensor -->
     <xacro:macro name="sensors" params="namespace sensor_name *origin">
-        <link name="ir_sensor/${sensor_name}">
+        <link name="${namespace}/ir_sensor/${sensor_name}">
             <inertial>
                 <origin
@@ -24,8 +25,8 @@
                 link="${namespace}/base_link"/>
             <child
-                link="ir_sensor/${sensor_name}"/>
+                link="${namespace}/ir_sensor/${sensor_name}"/>
             <xacro:insert_block name="origin"/>
         </joint>
-        <xacro:ir_sensor sensor_name="${sensor_name}"/>
+        <xacro:ir_sensor namespace="${namespace}" sensor_name="${sensor_name}"/>
     </xacro:macro>
 </robot>

File: urdf/doogie_wheels.xacro (robot description, xacro)
@@ -5,5 +5,5 @@
     <!-- macro: wheel -->
     <xacro:macro name="wheels" params="namespace wheel *mesh *origin *axis">
-    <link name="wheel/${wheel}">
+    <link name="${namespace}/wheel/${wheel}">
         <inertial>
             <origin
@@ -39,5 +39,5 @@
     <joint name="wheel/${wheel}_joint" type="continuous">
         <parent link="${namespace}/base_link"/>
-        <child link="wheel/${wheel}"/>
+        <child link="${namespace}/wheel/${wheel}"/>
         <xacro:insert_block name="origin"/>
         <xacro:insert_block name="axis"/>
