Commit message: Change wheel orientation based on axis parameter

File: urdf/doogie_wheels.xacro (robot description, xacro)
@@ -4,5 +4,5 @@
     <!--xacro:include filename="$(find doogie_description)/urdf/common_properties.xacro"/-->
     <!-- macro: wheel -->
-    <xacro:macro name="wheels" params="namespace sufix *mesh *joint_pose">
+    <xacro:macro name="wheels" params="namespace sufix *mesh *joint_pose *axis">
     <link name="wheel/${sufix}">
         <inertial>
@@ -35,5 +35,5 @@
         <child link="wheel/${sufix}"/>
         <xacro:insert_block name="joint_pose"/>
-        <axis xyz="-1 0 0"/>
+        <xacro:insert_block name="axis"/>
     </joint>
     <transmission name="wheel/${sufix}_trans" type="SimpleTransmission">
@@ -41,4 +41,5 @@
         <actuator name="$wheel/${sufix}_motor">
             <mechanicalReduction>1</mechanicalReduction>
+            <hardwareInterface>VelocityJointInterface</hardwareInterface>
         </actuator>
         <joint name="wheel/${sufix}_joint">

Commit message: Add friction to wheel joints

File: urdf/doogie_wheels.xacro (robot description, xacro)
@@ -36,4 +36,5 @@
         <xacro:insert_block name="joint_pose"/>
         <xacro:insert_block name="axis"/>
+        <dynamics friction="0.3"/>
     </joint>
     <transmission name="wheel/${sufix}_trans" type="SimpleTransmission">

Commit message: Update wheel to v3

File: urdf/doogie_wheels.xacro (robot description, xacro)
@@ -4,6 +4,6 @@
     <!--xacro:include filename="$(find doogie_description)/urdf/common_properties.xacro"/-->
     <!-- macro: wheel -->
-    <xacro:macro name="wheels" params="namespace wheel *mesh *origin *axis">
-    <link name="${namespace}/wheel/${wheel}">
+    <xacro:macro name="wheels" params="namespace wheel_name *mesh *origin *axis">
+    <link name="${namespace}/wheel/${wheel_name}">
         <inertial>
             <origin
@@ -37,18 +37,25 @@
         </collision>
     </link>
-    <joint name="wheel/${wheel}_joint" type="continuous">
-        <parent link="${namespace}/base_link"/>
-        <child link="${namespace}/wheel/${wheel}"/>
+    <joint name="wheel/${wheel_name}_joint" type="continuous">
+        <parent
+            link="${namespace}/base_link"/>
+        <child
+            link="${namespace}/wheel/${wheel_name}"/>
+        <dynamics
+            friction="0.3"/>
         <xacro:insert_block name="origin"/>
         <xacro:insert_block name="axis"/>
-        <dynamics friction="0.3"/>
     </joint>
-    <transmission name="wheel/${wheel}_trans" type="SimpleTransmission">
+    <transmission name="wheel/${wheel_name}_trans" type="SimpleTransmission">
         <type>transmission_interface/SimpleTransmission</type>
-        <actuator name="$wheel/${wheel}_motor">
+        <actuator name="wheel/${wheel_name}_motor">
             <mechanicalReduction>1</mechanicalReduction>
+            <!--
+                The hardwareInterface tag is optional, but is used here to maintain compatibility
+                with ROS releases prior to Indigo.
+            -->
             <hardwareInterface>VelocityJointInterface</hardwareInterface>
         </actuator>
-        <joint name="wheel/${wheel}_joint">
+        <joint name="wheel/${wheel_name}_joint">
             <hardwareInterface>hardware_interface/VelocityJointInterface</hardwareInterface>
         </joint>
