Commit message: Add package configuration files

File: urdf/doogie.urdf.xacro (robot description, xacro)
@@ -1,3 +1,9 @@
 <?xml version="1.0"?>
 <robot name="doogie" xmlns:xacro="http://www.ros.org/wiki/xacro">
+    <!-- Parameters -->
+    <xacro:arg name="namespace" default="doogie"/>
+    <!-- Includes -->
+    <xacro:include filename="$(find doogie_description)/urdf/doogie_base.xacro"/>
+    <!-- Creates the doogie -->
+    <xacro:doogie_base namespace="$(arg namespace)"/>
 </robot>

File: urdf/doogie_base.xacro (robot description, xacro)
@@ -1,7 +1,10 @@
 <?xml version="1.0"?>
 <robot xmlns:xacro="http://www.ros.org/wiki/xacro">
-    <xacro:property name="mass" value="2.5">
+    <!-- Parameters -->
+    <xacro:property name="mass" value="2.5"/>
+    <xacro:property name="namespace" value="doogie"/>
+    <!-- macro: base -->
     <xacro:macro name="doogie_base" params="namespace">
-        <link name="link_name">
+        <link name="${namespace}/link_name">
             <inertial>
                 <origin xyz="0 0 0" rpy="0 0 0"/>
@@ -12,5 +15,5 @@
                 <origin xyz="0 0 0" rpy="0 0 0"/>
                 <geometry>
-                    <box size="0.10 0.3 0.5"/>
+                    <box size="0.5 0.3 0.1"/>
                 </geometry>
             </visual>
@@ -18,7 +21,8 @@
                 <origin xyz="0 0 0" rpy="0 0 0"/>
                 <geometry>
-                    <box size="0.10 0.3 0.5"/>
+                    <box size="0.5 0.3 0.1"/>
                 </geometry>
             </collision>
         </link>
+    </xacro:macro>
 </robot>

Commit message: Change xmlns:xacro to new model

File: urdf/doogie.urdf.xacro (robot description, xacro)
@@ -1,9 +1,24 @@
 <?xml version="1.0"?>
-<robot name="doogie" xmlns:xacro="http://www.ros.org/wiki/xacro">
+<robot name="doogie" xmlns:xacro="http://ros.org/wiki/xacro">
     <!-- Parameters -->
     <xacro:arg name="namespace" default="doogie"/>
     <!-- Includes -->
+    <xacro:include filename="$(find doogie_description)/urdf/common_properties.xacro"/>
     <xacro:include filename="$(find doogie_description)/urdf/doogie_base.xacro"/>
-    <!-- Creates the doogie -->
+    <xacro:include filename="$(find doogie_description)/urdf/doogie_wheels.xacro"/>
+    <!-- Creates doogie base -->
     <xacro:doogie_base namespace="$(arg namespace)"/>
+    <!-- Creates wheels -->
+    <xacro:wheels namespace="$(arg namespace)" sufix="front_left">
+         <origin xyz="0 0.3 0" rpy="0 0 0" />
+    </xacro:wheels>
+    <xacro:wheels namespace="$(arg namespace)" sufix="front_right">
+        <origin xyz="0 0 0" rpy="0 0 0" />
+    </xacro:wheels>
+    <xacro:wheels namespace="$(arg namespace)" sufix="rear_left">
+        <origin xyz="0 0 0" rpy="0 0 0" />
+    </xacro:wheels>
+    <xacro:wheels namespace="$(arg namespace)" sufix="rear_right">
+        <origin xyz="0 0 0" rpy="0 0 0" />
+    </xacro:wheels>
 </robot>

File: urdf/doogie_base.xacro (robot description, xacro)
@@ -1,10 +1,12 @@
 <?xml version="1.0"?>
-<robot xmlns:xacro="http://www.ros.org/wiki/xacro">
+<robot xmlns:xacro="http://ros.org/wiki/xacro">
     <!-- Parameters -->
     <xacro:property name="mass" value="2.5"/>
     <xacro:property name="namespace" value="doogie"/>
+    <!-- Includes -->
+    <!-- xacro:include filename="$(find doogie_description)/urdf/common_properties.xacro"/ -->
     <!-- macro: base -->
     <xacro:macro name="doogie_base" params="namespace">
-        <link name="${namespace}/link_name">
+        <link name="${namespace}/base_link">
             <inertial>
                 <origin xyz="0 0 0" rpy="0 0 0"/>
@@ -17,4 +19,5 @@
                     <box size="0.5 0.3 0.1"/>
                 </geometry>
+                <material name="red"/>
             </visual>
             <collision>

Commit message: Add meshes to urdf and transmission informations

File: urdf/doogie.urdf.xacro (robot description, xacro)
@@ -10,15 +10,17 @@
     <xacro:doogie_base namespace="$(arg namespace)"/>
     <!-- Creates wheels -->
-    <xacro:wheels namespace="$(arg namespace)" sufix="front_left">
-         <origin xyz="0 0.3 0" rpy="0 0 0" />
+    <xacro:wheels namespace="$(arg namespace)" sufix="left">
+        <mesh
+          filename="package://doogie_description/meshes/collada/wheel.dae" />
+        <origin
+          xyz="-0.011296 0.044721 0.00521"
+          rpy="1.6313 0 -1.5708" />
     </xacro:wheels>
-    <xacro:wheels namespace="$(arg namespace)" sufix="front_right">
-        <origin xyz="0 0 0" rpy="0 0 0" />
-    </xacro:wheels>
-    <xacro:wheels namespace="$(arg namespace)" sufix="rear_left">
-        <origin xyz="0 0 0" rpy="0 0 0" />
-    </xacro:wheels>
-    <xacro:wheels namespace="$(arg namespace)" sufix="rear_right">
-        <origin xyz="0 0 0" rpy="0 0 0" />
+    <xacro:wheels namespace="$(arg namespace)" sufix="right">
+        <mesh
+          filename="package://doogie_description/meshes/collada/wheel.dae" />
+        <origin
+          xyz="-0.011296 -0.044079 0.00521"
+          rpy="-1.6313 0 1.5708" />
     </xacro:wheels>
 </robot>

File: urdf/doogie_base.xacro (robot description, xacro)
@@ -2,5 +2,5 @@
 <robot xmlns:xacro="http://ros.org/wiki/xacro">
     <!-- Parameters -->
-    <xacro:property name="mass" value="2.5"/>
+    <xacro:property name="mass" value="0.029195"/>
     <xacro:property name="namespace" value="doogie"/>
     <!-- Includes -->
@@ -10,19 +10,24 @@
         <link name="${namespace}/base_link">
             <inertial>
-                <origin xyz="0 0 0" rpy="0 0 0"/>
+                <origin xyz="0.0022635 0.00032106 0.00030753" rpy="0 0 0"/>
                 <mass value="${mass}"/>
-                <inertia ixx="0.0001" ixy="0.0001" ixz="0.0001" iyy="0.0001" iyz="0.0001" izz="0.0001"/>
+                <inertia
+                    ixx="1.2452E-05"
+                    ixy="3.9492E-12"
+                    ixz="8.5399E-17"
+                    iyy="1.635E-05"
+                    iyz="7.6951E-15"
+                    izz="2.8634E-05" />
             </inertial>
-            <visual name="">
+            <visual>
                 <origin xyz="0 0 0" rpy="0 0 0"/>
                 <geometry>
-                    <box size="0.5 0.3 0.1"/>
+                    <mesh filename="package://doogie_description/meshes/collada/base.dae"/>
                 </geometry>
-                <material name="red"/>
             </visual>
             <collision>
                 <origin xyz="0 0 0" rpy="0 0 0"/>
                 <geometry>
-                    <box size="0.5 0.3 0.1"/>
+                    <mesh filename="package://doogie_description/meshes/collada/base.dae"/>
                 </geometry>
             </collision>

File: urdf/doogie_wheels.xacro (robot description, xacro)
@@ -4,15 +4,21 @@
     <!--xacro:include filename="$(find doogie_description)/urdf/common_properties.xacro"/-->
     <!-- macro: wheel -->
-    <xacro:macro name="wheels" params="namespace sufix *joint_pose">
+    <xacro:macro name="wheels" params="namespace sufix *mesh *joint_pose">
     <link name="wheel/${sufix}">
         <inertial>
-            <origin xyz="0.0 0.0 0.0" rpy="0.0 0.0 0.0"/>
-            <mass value="2.6"/>
-            <inertia ixx="0.02467" ixy="0" ixz="0" iyy="0.04411" iyz="0" izz="0.02467"/>
+            <origin xyz="0.0033664 1.419E-05 -1.7243E-07" rpy="0.0 0.0 0.0"/>
+            <mass value="0.0029447"/>
+            <inertia
+              ixx="4.567E-07"
+              ixy="4.239E-11"
+              ixz="-5.3853E-13"
+              iyy="2.3874E-07"
+              iyz="-1.5273E-12"
+              izz="2.3862E-07" />
         </inertial>
         <visual>
             <origin xyz="0.0 0.0 0.0" rpy="0.0 0.0 0.0"/>
             <geometry>
-                <cylinder length="0.008" radius="0.046"/>
+                <xacro:insert_block name="mesh"/>
             </geometry>
             <material name="dark"/>
@@ -21,23 +27,23 @@
             <origin xyz="0.0 0.0 0.0" rpy="0.0 0.0 0.0"/>
             <geometry>
-                <cylinder length="0.008" radius="0.046"/>
+                <xacro:insert_block name="mesh"/>
             </geometry>
         </collision>
     </link>
-    <gazebo reference="wheel/${sufix}_link">
-        <material>Gazebo/DarkGrey</material>
-        <selfCollide>false</selfCollide>
-        <mu1 value="0.5"/>
-        <mu2 value="0.5"/>
-        <kp value="10000000.0" />
-        <kd value="1" />
-        <fdir1 value="1 0 0"/>
-    </gazebo>
     <joint name="wheel/${sufix}_joint" type="continuous">
         <parent link="${namespace}/base_link"/>
         <child link="wheel/${sufix}"/>
         <xacro:insert_block name="joint_pose"/>
-        <axis xyz="0 0 0"/>
+        <axis xyz="-1 0 0"/>
     </joint>
+    <transmission name="wheel/${sufix}_trans" type="SimpleTransmission">
+        <type>transmission_interface/SimpleTransmission</type>
+        <actuator name="$wheel/${sufix}_motor">
+            <mechanicalReduction>1</mechanicalReduction>
+        </actuator>
+        <joint name="wheel/${sufix}_joint">
+            <hardwareInterface>hardware_interface/VelocityJointInterface</hardwareInterface>
+        </joint>
+    </transmission>
     </xacro:macro>
 </robot>

Commit message: Add ros_control gazebo plugin to doogie_urdf and some more minor fixes

File: urdf/doogie.urdf.xacro (robot description, xacro)
@@ -16,4 +16,6 @@
           xyz="-0.011296 0.044721 0.00521"
           rpy="1.6313 0 -1.5708" />
+        <axis
+          xyz="-1.0 0.0 0.0"/>
     </xacro:wheels>
     <xacro:wheels namespace="$(arg namespace)" sufix="right">
@@ -23,4 +25,6 @@
           xyz="-0.011296 -0.044079 0.00521"
           rpy="-1.6313 0 1.5708" />
+        <axis
+          xyz="1.0 0.0 0.0"/>
     </xacro:wheels>
     <gazebo>

Commit message: Change 'sufix' to 'wheel' in doogie_wheels.xacro

File: urdf/doogie.urdf.xacro (robot description, xacro)
@@ -10,25 +10,25 @@
     <xacro:doogie_base namespace="$(arg namespace)"/>
     <!-- Creates wheels -->
-    <xacro:wheels namespace="$(arg namespace)" sufix="left">
+    <xacro:wheels namespace="$(arg namespace)" wheel="left">
         <mesh
-          filename="package://doogie_description/meshes/collada/wheel.dae" />
+            filename="package://doogie_description/meshes/collada/wheel.dae" />
         <origin
-          xyz="-0.011296 0.044721 0.00521"
-          rpy="1.6313 0 -1.5708" />
+            xyz="-0.011296 0.044721 0.00521"
+            rpy="1.6313 0 -1.5708" />
         <axis
-          xyz="-1.0 0.0 0.0"/>
+            xyz="-1.0 0.0 0.0"/>
     </xacro:wheels>
-    <xacro:wheels namespace="$(arg namespace)" sufix="right">
+    <xacro:wheels namespace="$(arg namespace)" wheel="right">
         <mesh
-          filename="package://doogie_description/meshes/collada/wheel.dae" />
+            filename="package://doogie_description/meshes/collada/wheel.dae" />
         <origin
-          xyz="-0.011296 -0.044079 0.00521"
-          rpy="-1.6313 0 1.5708" />
+            xyz="-0.011296 -0.044079 0.00521"
+            rpy="-1.6313 0 1.5708" />
         <axis
-          xyz="1.0 0.0 0.0"/>
+            xyz="1.0 0.0 0.0"/>
     </xacro:wheels>
     <gazebo>
     <plugin name="gazebo_ros_control" filename="libgazebo_ros_control.so">
-      <robotNamespace>$(arg namespace)</robotNamespace>
+        <robotNamespace>$(arg namespace)</robotNamespace>
     </plugin>
     </gazebo>

File: urdf/doogie_wheels.xacro (robot description, xacro)
@@ -4,19 +4,24 @@
     <!--xacro:include filename="$(find doogie_description)/urdf/common_properties.xacro"/-->
     <!-- macro: wheel -->
-    <xacro:macro name="wheels" params="namespace sufix *mesh *joint_pose *axis">
-    <link name="wheel/${sufix}">
+    <xacro:macro name="wheels" params="namespace wheel *mesh *joint_pose *axis">
+    <link name="wheel/${wheel}">
         <inertial>
-            <origin xyz="0.0033664 1.419E-05 -1.7243E-07" rpy="0.0 0.0 0.0"/>
-            <mass value="0.0029447"/>
+            <origin
+                xyz="0.0033664 1.419E-05 -1.7243E-07"
+                rpy="0.0 0.0 0.0"/>
+            <mass
+                value="0.0029447"/>
             <inertia
-              ixx="4.567E-07"
-              ixy="4.239E-11"
-              ixz="-5.3853E-13"
-              iyy="2.3874E-07"
-              iyz="-1.5273E-12"
-              izz="2.3862E-07" />
+                ixx="4.567E-07"
+                ixy="4.239E-11"
+                ixz="-5.3853E-13"
+                iyy="2.3874E-07"
+                iyz="-1.5273E-12"
+                izz="2.3862E-07" />
         </inertial>
         <visual>
-            <origin xyz="0.0 0.0 0.0" rpy="0.0 0.0 0.0"/>
+            <origin
+                xyz="0.0 0.0 0.0"
+                rpy="0.0 0.0 0.0"/>
             <geometry>
                 <xacro:insert_block name="mesh"/>
@@ -25,5 +30,7 @@
         </visual>
         <collision>
-            <origin xyz="0.0 0.0 0.0" rpy="0.0 0.0 0.0"/>
+            <origin
+                xyz="0.0 0.0 0.0"
+                rpy="0.0 0.0 0.0"/>
             <geometry>
                 <xacro:insert_block name="mesh"/>
@@ -31,18 +38,18 @@
         </collision>
     </link>
-    <joint name="wheel/${sufix}_joint" type="continuous">
+    <joint name="wheel/${wheel}_joint" type="continuous">
         <parent link="${namespace}/base_link"/>
-        <child link="wheel/${sufix}"/>
+        <child link="wheel/${wheel}"/>
         <xacro:insert_block name="joint_pose"/>
         <xacro:insert_block name="axis"/>
         <dynamics friction="0.3"/>
     </joint>
-    <transmission name="wheel/${sufix}_trans" type="SimpleTransmission">
+    <transmission name="wheel/${wheel}_trans" type="SimpleTransmission">
         <type>transmission_interface/SimpleTransmission</type>
-        <actuator name="$wheel/${sufix}_motor">
+        <actuator name="$wheel/${wheel}_motor">
             <mechanicalReduction>1</mechanicalReduction>
             <hardwareInterface>VelocityJointInterface</hardwareInterface>
         </actuator>
-        <joint name="wheel/${sufix}_joint">
+        <joint name="wheel/${wheel}_joint">
             <hardwareInterface>hardware_interface/VelocityJointInterface</hardwareInterface>
         </joint>

Commit message: Add ir_sensor to doogie_sensors.xacro

File: urdf/doogie.urdf.xacro (robot description, xacro)
@@ -7,7 +7,8 @@
     <xacro:include filename="$(find doogie_description)/urdf/doogie_base.xacro"/>
     <xacro:include filename="$(find doogie_description)/urdf/doogie_wheels.xacro"/>
-    <!-- Creates doogie base -->
+    <xacro:include filename="$(find doogie_description)/urdf/doogie_sensors.xacro"/>
+    <!-- Create doogie base -->
     <xacro:doogie_base namespace="$(arg namespace)"/>
-    <!-- Creates wheels -->
+    <!-- Create wheels -->
     <xacro:wheels namespace="$(arg namespace)" wheel="left">
         <mesh
@@ -28,8 +29,30 @@
             xyz="1.0 0.0 0.0"/>
     </xacro:wheels>
+    <!-- Add ros_control plugin -->
     <gazebo>
-    <plugin name="gazebo_ros_control" filename="libgazebo_ros_control.so">
-        <robotNamespace>$(arg namespace)</robotNamespace>
-    </plugin>
+        <plugin name="gazebo_ros_control" filename="libgazebo_ros_control.so">
+            <robotNamespace>$(arg namespace)</robotNamespace>
+        </plugin>
     </gazebo>
+    <!-- Create ir_sensors -->
+    <xacro:sensors namespace="$(arg namespace)" sensor_name="left">
+        <origin
+            xyz="0.0364324038765062 0.0351454111038035 -0.01074"
+            rpy="1.5707963267949 0 0.17453"/>
+    </xacro:sensors>
+    <xacro:sensors namespace="$(arg namespace)" sensor_name="front_left">
+        <origin
+            xyz="0.052482 0.014629 -0.01074"
+            rpy="1.5707963267949 0 0.87266"/>
+    </xacro:sensors>
+    <xacro:sensors namespace="$(arg namespace)" sensor_name="front_right">
+        <origin
+            xyz="0.0524823992514108 -0.0146287488616027 -0.01074"
+            rpy="1.5707963267949 0 -0.87266"/>
+    </xacro:sensors>
+    <xacro:sensors namespace="$(arg namespace)" sensor_name="right">
+        <origin
+            xyz="0.036432 -0.035145 -0.01074"
+            rpy="1.5708 0 -0.17453"/>
+    </xacro:sensors>
 </robot>

File: urdf/doogie_base.xacro (robot description, xacro)
@@ -2,5 +2,5 @@
 <robot xmlns:xacro="http://ros.org/wiki/xacro">
     <!-- Parameters -->
-    <xacro:property name="mass" value="0.029195"/>
+    <xacro:property name="mass" value="0.03293"/>
     <xacro:property name="namespace" value="doogie"/>
     <!-- Includes -->
@@ -10,18 +10,21 @@
         <link name="${namespace}/base_link">
             <inertial>
-                <origin xyz="0.0022635 0.00032106 0.00030753" rpy="0 0 0"/>
-                <mass value="${mass}"/>
+                <origin
+                    xyz="0.00968674071529441 -4.2987819602154E-18 -0.0125192407288749"
+                    rpy="0 0 0"/>
+                <mass
+                    value="${mass}"/>
                 <inertia
-                    ixx="1.2452E-05"
-                    ixy="3.9492E-12"
-                    ixz="8.5399E-17"
-                    iyy="1.635E-05"
-                    iyz="7.6951E-15"
-                    izz="2.8634E-05" />
+                    ixx="1.52668608193465E-05"
+                    ixy="4.58917710661775E-12"
+                    ixz="2.73567369382039E-23"
+                    iyy="1.93599497928914E-05"
+                    iyz="-2.31610571514848E-23"
+                    izz="3.44511538963699E-05" />
             </inertial>
             <visual>
                 <origin xyz="0 0 0" rpy="0 0 0"/>
                 <geometry>
-                    <mesh filename="package://doogie_description/meshes/collada/base.dae"/>
+                    <mesh filename="package://doogie_description/meshes/collada/base_link_v3.dae"/>
                 </geometry>
             </visual>
@@ -29,5 +32,5 @@
                 <origin xyz="0 0 0" rpy="0 0 0"/>
                 <geometry>
-                    <mesh filename="package://doogie_description/meshes/collada/base.dae"/>
+                    <mesh filename="package://doogie_description/meshes/collada/base_link_v3.dae"/>
                 </geometry>
             </collision>

File: urdf/doogie_wheels.xacro (robot description, xacro)
@@ -4,5 +4,5 @@
     <!--xacro:include filename="$(find doogie_description)/urdf/common_properties.xacro"/-->
     <!-- macro: wheel -->
-    <xacro:macro name="wheels" params="namespace wheel *mesh *joint_pose *axis">
+    <xacro:macro name="wheels" params="namespace wheel *mesh *origin *axis">
     <link name="wheel/${wheel}">
         <inertial>
@@ -41,5 +41,5 @@
         <parent link="${namespace}/base_link"/>
         <child link="wheel/${wheel}"/>
-        <xacro:insert_block name="joint_pose"/>
+        <xacro:insert_block name="origin"/>
         <xacro:insert_block name="axis"/>
         <dynamics friction="0.3"/>

Commit message: Change wheel meshes to collada version

File: urdf/doogie.urdf.xacro (robot description, xacro)
@@ -13,5 +13,5 @@
     <xacro:wheels namespace="$(arg namespace)" wheel="left">
         <mesh
-            filename="package://doogie_description/meshes/stl/left_wheel.STL" />
+            filename="package://doogie_description/meshes/collada/wheel_v3.dae" />
         <origin
             xyz="0.00302 0.0464 -0.00444"
@@ -22,5 +22,5 @@
     <xacro:wheels namespace="$(arg namespace)" wheel="right">
         <mesh
-            filename="package://doogie_description/meshes/stl/left_wheel.STL" />
+            filename="package://doogie_description/meshes/collada/wheel_v3.dae" />
         <origin
             xyz="0.00302 -0.0464 -0.00444"

File: urdf/doogie_wheels.xacro (robot description, xacro)
@@ -27,5 +27,4 @@
                 <xacro:insert_block name="mesh"/>
             </geometry>
-            <material name="dark"/>
         </visual>
         <collision>

Commit message: Update doogie_urdf to v0.4

File: urdf/doogie.urdf.xacro (robot description, xacro)
@@ -11,21 +11,21 @@
     <xacro:doogie_base namespace="$(arg namespace)"/>
     <!-- Create wheels -->
-    <xacro:wheels namespace="$(arg namespace)" wheel="left">
+    <xacro:wheels namespace="$(arg namespace)" wheel_name="left">
         <mesh
-            filename="package://doogie_description/meshes/collada/wheel_v3.dae" />
+            filename="package://doogie_description/meshes/collada/wheel_v3.dae"/>
         <origin
             xyz="0.00302 0.0464 -0.00444"
-            rpy="1.5708 0 1.5708" />
+            rpy="1.5708 0 1.5708"/>
+        <axis
+            xyz="1.0 0.0 0.0"/>
+    </xacro:wheels>
+    <xacro:wheels namespace="$(arg namespace)" wheel_name="right">
+        <mesh
+            filename="package://doogie_description/meshes/collada/wheel_v3.dae"/>
+        <origin
+            xyz="0.00302 -0.0464 -0.00444"
+            rpy="1.5708 0 -1.5708"/>
         <axis
             xyz="-1.0 0.0 0.0"/>
-    </xacro:wheels>
-    <xacro:wheels namespace="$(arg namespace)" wheel="right">
-        <mesh
-            filename="package://doogie_description/meshes/collada/wheel_v3.dae" />
-        <origin
-            xyz="0.00302 -0.0464 -0.00444"
-            rpy="1.5708 0 -1.5708" />
-        <axis
-            xyz="1.0 0.0 0.0"/>
     </xacro:wheels>
     <!-- Add ros_control plugin -->
