Commit message: Add different names for each ir_sensor

File: urdf/acessories/ir_sensor.xacro (robot description, xacro)
@@ -1,7 +1,7 @@
 <?xml version="1.0"?>
 <robot xmlns:xacro="http://ros.org/wiki/xacro">
-    <xacro:macro name="ir_sensor" params="sensor_name">
-        <gazebo reference="ir_sensor/${sensor_name}">
-         <sensor type="ray" name="head_hokuyo_sensor">
+    <xacro:macro name="ir_sensor" params="namespace sensor_name">
+        <gazebo reference="${namespace}/ir_sensor/${sensor_name}">
+         <sensor type="ray" name="${sensor_name}">
             <pose>0 0 0 0 0 0</pose>
             <visualize>true</visualize>
@@ -15,10 +15,4 @@
                      <max_angle>0.14835</max_angle>
                   </horizontal>
-                  <vertical>
-                     <samples>70</samples>
-                     <resolution>1</resolution>
-                     <min_angle>-0.14835</min_angle>
-                     <max_angle>0.14835</max_angle>
-                  </vertical>
                </scan>
                <range>
