Commit message: Update minus maze meshes optimazing it

File: mazes/minus.urdf (robot description, URDF)
Before this commit: robot minus_maze, 1 links, 0 joints
Links:
- link minus/base_link: geometry collision mesh filename=package://doogie_description/mazes/minus_collision.dae; visual mesh filename=package://doogie_description/mazes/minus_visual.dae
