Commit message: Update Minus maze model

File: doogie_description/mazes/minus.urdf (robot description, URDF)
Before this commit: robot minus_maze, 1 links, 0 joints
Links:
- link minus/base_link: geometry collision mesh filename=package://doogie_description/mazes/minus_collision.dae; visual mesh filename=package://doogie_description/mazes/minus_visual_v2.dae

Commit message: Change mesh's names suffixes

File: doogie_description/mazes/minus.urdf (robot description, URDF)
Before this commit: robot minus_maze, 1 links, 0 joints
Links:
- link minus/base_link: geometry collision mesh filename=package://doogie_description/mazes/minus_collision.dae; visual mesh filename=package://doogie_description/mazes/minus_visual.dae

File: doogie_description/urdf/doogie.urdf.xacro (robot description, xacro)
@@ -14,5 +14,5 @@
     <xacro:wheels namespace="$(arg namespace)" wheel_name="left">
         <mesh
-            filename="package://doogie_description/meshes/collada/wheel_v3.dae"/>
+            filename="package://doogie_description/meshes/collada/wheel.dae"/>
         <origin
             xyz="0.00302 0.0464 -0.00444"
@@ -23,5 +23,5 @@
     <xacro:wheels namespace="$(arg namespace)" wheel_name="right">
         <mesh
-            filename="package://doogie_description/meshes/collada/wheel_v3.dae"/>
+            filename="package://doogie_description/meshes/collada/wheel.dae"/>
         <origin
             xyz="0.00302 -0.0464 -0.00444"

File: doogie_description/urdf/doogie_base.xacro (robot description, xacro)
@@ -28,5 +28,5 @@
                 rpy="0 0 0"/>
             <geometry>
-                <mesh filename="package://doogie_description/meshes/collada/base_link_v4.dae"/>
+                <mesh filename="package://doogie_description/meshes/collada/base_link.dae"/>
             </geometry>
         </visual>

Commit message: Fix maze visual mesh

File: doogie_description/mazes/minus.urdf (robot description, URDF)
Before this commit: robot minus_maze, 1 links, 0 joints
Links:
- link minus/base_link: geometry collision box size=0.03 0.03 0.001; collision mesh filename=package://doogie_description/mazes/minus_collision.stl
