Commit message: Update robot model to optimize its collision box

File: doogie_description/urdf/doogie_base.xacro (robot description, xacro)
@@ -36,5 +36,13 @@
                 rpy="0 0 0"/>
             <geometry>
-                <mesh filename="package://doogie_description/meshes/collada/base_link_v4.dae"/>
+                <mesh filename="package://doogie_description/meshes/stl/doogie_collision.stl"/>
+            </geometry>
+        </collision>
+        <collision>
+            <origin
+                xyz="0.063 0 -0.018"
+                rpy="0 0 0"/>
+            <geometry>
+                <box size="0.005 0.005 -0.005"/>
             </geometry>
         </collision>

File: doogie_description/urdf/doogie_wheels.xacro (robot description, xacro)
@@ -30,9 +30,9 @@
         <collision>
             <origin
-                xyz="0.0 0.0 0.0"
-                rpy="0.0 0.0 0.0"/>
+                xyz="-0.0025 0.0 0.0"
+                rpy="0.0 1.5708 0.0"/>
             <geometry>
-                <xacro:insert_block name="mesh"/>
-            </geometry>
+                <cylinder radius="0.0162" length="0.005"/>
+             </geometry>
         </collision>
     </link>

Commit message: Add kinematics gazebo parameters to stop robot moving by itself

File: doogie_description/urdf/doogie_base.xacro (robot description, xacro)
@@ -44,5 +44,5 @@
                 rpy="0 0 0"/>
             <geometry>
-                <box size="0.005 0.005 -0.005"/>
+                <box size="0.005 0.005 -0.0065"/>
             </geometry>
         </collision>

File: doogie_description/urdf/doogie_wheels.xacro (robot description, xacro)
@@ -33,5 +33,5 @@
                 rpy="0.0 1.5708 0.0"/>
             <geometry>
-                <cylinder radius="0.0162" length="0.005"/>
+                <cylinder radius="0.0177" length="0.005"/>
              </geometry>
         </collision>
@@ -43,5 +43,5 @@
             link="${namespace}/wheel/${wheel_name}"/>
         <dynamics
-            friction="0.3"/>
+            friction="0.6"/>
         <xacro:insert_block name="origin"/>
         <xacro:insert_block name="axis"/>
@@ -61,4 +61,12 @@
         </joint>
     </transmission>
+    <gazebo reference="${namespace}/wheel/${wheel_name}">
+        <kp>1000000.0</kp>
+        <kd>100.0</kd>
+        <mu1>1.0</mu1>
+        <mu2>1.0</mu2>
+        <maxVel>0.5</maxVel>
+        <minDepth>0.0005</minDepth>
+    </gazebo>
     </xacro:macro>
 </robot>
