Commit message: Fix robot's kinematics

File: doogie_description/urdf/doogie.urdf.xacro (robot description, xacro)
@@ -30,12 +30,40 @@
             xyz="-1.0 0.0 0.0"/>
     </xacro:wheels>
-    <!-- Add ros_control plugin -->
+    <!-- Model Plugins -->
     <gazebo>
+        <!-- ros_control plugin -->
         <plugin name="gazebo_ros_control" filename="libgazebo_ros_control.so">
-        <!-- robotnamespace tag is note used here because it
+        <!-- robotnamespace tag is not used here because it
              blocks changing robot namespace in extern launchfiles
          -->
             <robotParam>$(arg robotParam)</robotParam>
         </plugin>
+        <!-- ground truth plugin -->
+        <plugin name="gazebo_ros_p3d" filename="libgazebo_ros_p3d.so">
+            <alwaysOn>true</alwaysOn>
+            <updateRate>100.0</updateRate>
+            <bodyName>$(arg namespace)/base_link</bodyName>
+            <topicName>/gazebo/ground_truth</topicName>
+            <!-- <frameName>world</frameName> -->
+            <!-- <gaussianNoise>0.0</gaussianNoise>
+            <xyzOffsets>0 0 0</xyzOffsets>
+            <rpyOffsets>0 0 0</rpyOffsets> -->
+        </plugin>
+    </gazebo>
+    <!--  Add colision sensor plugin -->
+    <gazebo reference="$(arg namespace)/base_link">
+        <sensor name="bumper_sensor" type="contact">
+            <always_on>true</always_on>
+            <update_rate>1</update_rate>
+            <contact>
+                <collision>/base_link_fixed_joint_lump__doogie_collision_collision</collision>
+            </contact>
+            <plugin name="gazebo_ros_bumper" filename="libgazebo_ros_bumper.so">
+                <bumperTopicName>bumper</bumperTopicName>
+                <frameName>base_link</frameName>
+                <always_on>true</always_on>
+                <update_rate>1</update_rate>
+            </plugin>
+        </sensor>
     </gazebo>
     <!-- Create ir_sensors -->

File: doogie_description/urdf/doogie_base.xacro (robot description, xacro)
@@ -2,5 +2,5 @@
 <robot xmlns:xacro="http://ros.org/wiki/xacro">
     <!-- Parameters -->
-    <xacro:property name="mass" value="0.03293"/>
+    <xacro:property name="mass" value="10.0"/>
     <xacro:property name="namespace" value="doogie"/>
     <!-- Includes -->
@@ -11,28 +11,28 @@
         <inertial>
             <origin
-                xyz="0.00968674071529441 -4.2987819602154E-18 -0.0125192407288749"
+                xyz="0.0247 0.0 -0.0125"
                 rpy="0 0 0"/>
             <mass
                 value="${mass}"/>
             <inertia
-                ixx="1.52668608193465E-05"
-                ixy="4.58917710661775E-12"
-                ixz="2.73567369382039E-23"
-                iyy="1.93599497928914E-05"
-                iyz="-2.31610571514848E-23"
-                izz="3.44511538963699E-05" />
+                ixx="10"
+                ixy="0"
+                ixz="0"
+                iyy="10"
+                iyz="0"
+                izz="10"/>
         </inertial>
         <visual>
             <origin
-                xyz="0 0 0"
-                rpy="0 0 0"/>
+                xyz="0.0 0.0 0.0"
+                rpy="0.0 0.0 0.0"/>
             <geometry>
                 <mesh filename="package://doogie_description/meshes/collada/base_link.dae"/>
             </geometry>
         </visual>
-        <collision>
+        <collision name="doogie_collision">
             <origin
-                xyz="0 0 0"
-                rpy="0 0 0"/>
+                xyz="0.0 0.0 0.0"
+                rpy="0.0 0.0 0.0"/>
             <geometry>
                 <mesh filename="package://doogie_description/meshes/stl/doogie_collision.stl"/>
@@ -41,15 +41,18 @@
         <collision>
             <origin
-                xyz="0.063 0 -0.018"
-                rpy="0 0 0"/>
+                xyz="0.063 0.0 -0.018"
+                rpy="0.0 0.0 0.0"/>
             <geometry>
-                <box size="0.005 0.005 -0.0065"/>
+                <box size="0.005 0.005 -0.0038"/>
             </geometry>
         </collision>
     </link>
-        <gazebo reference="${namespace}/base_link">
-            <kp>10000000</kp>
-            <kd>1</kd>
-        </gazebo>
+    <gazebo reference="${namespace}/base_link">
+        <dampingFactor>0.0025</dampingFactor>
+        <kp>1000000.0</kp>
+        <kd>1.0</kd>
+        <mu1>0.0</mu1>
+        <mu2>0.0</mu2>
+    </gazebo>
     </xacro:macro>
 </robot>

File: doogie_description/urdf/doogie_wheels.xacro (robot description, xacro)
@@ -11,12 +11,12 @@
                 rpy="0.0 0.0 0.0"/>
             <mass
-                value="0.0029447"/>
+                value="0.29447"/>
             <inertia
-                ixx="4.567E-07"
-                ixy="4.239E-11"
-                ixz="-5.3853E-13"
-                iyy="2.3874E-07"
-                iyz="-1.5273E-12"
-                izz="2.3862E-07" />
+                ixx="0.2"
+                ixy="0"
+                ixz="0"
+                iyy="0.2"
+                iyz="0"
+                izz="0.2" />
         </inertial>
         <visual>
@@ -33,5 +33,5 @@
                 rpy="0.0 1.5708 0.0"/>
             <geometry>
-                <cylinder radius="0.0177" length="0.005"/>
+                <cylinder radius="0.015" length="0.005"/>
              </geometry>
         </collision>
@@ -43,5 +43,6 @@
             link="${namespace}/wheel/${wheel_name}"/>
         <dynamics
-            friction="0.6"/>
+            friction="0.6"
+            damping="10.0"/>
         <xacro:insert_block name="origin"/>
         <xacro:insert_block name="axis"/>
@@ -50,5 +51,5 @@
         <type>transmission_interface/SimpleTransmission</type>
         <actuator name="wheel/${wheel_name}_motor">
-            <mechanicalReduction>1</mechanicalReduction>
+            <mechanicalReduction>2</mechanicalReduction>
             <!--
                 The hardwareInterface tag in below is optional when inside <actuator>, but it is used here to maintain compatibility
@@ -63,9 +64,21 @@
     <gazebo reference="${namespace}/wheel/${wheel_name}">
         <kp>1000000.0</kp>
-        <kd>100.0</kd>
-        <mu1>1.0</mu1>
-        <mu2>1.0</mu2>
+        <kd>1000.0</kd>
+        <mu1>5.0</mu1>
+        <mu2>5.0</mu2>
         <maxVel>0.5</maxVel>
-        <minDepth>0.0005</minDepth>
+        <!-- <minDepth>0.0005</minDepth> -->
+        <selfCollide>false</selfCollide>
+    </gazebo>
+    <gazebo reference="wheel/${wheel_name}_joint">
+        <provideFeedback>true</provideFeedback>
+        <!-- <implicitSpringDamper>true</implicitSpringDamper> -->
+    </gazebo>
+    <gazebo>
+      <plugin name="ft_sensor" filename="libgazebo_ros_ft_sensor.so">
+        <updateRate>1</updateRate>
+        <topicName>wheel/${wheel_name}_joint/ft_sensor_topic</topicName>
+        <jointName>wheel/${wheel_name}_joint</jointName>
+      </plugin>
     </gazebo>
     </xacro:macro>
